File: hardware/wFM-Tx_0.1/wFM-Tx_0.1.kicad_pcb (KiCad board)
At the start: 2 copper layers, 53.2 x 40.3 mm, 27 parts, among them P1 1x3, P2 1x2, P3 1x2, P4 1x6, P5 2x3, P6 1x3, Q1 MMBT3904, Q2 MMBT3904, SW1 EG2219, U1 ATmega328P-AU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

Commit message: Added silkscreen text on PCB, updated gerbers
Parts:
- added SYM0: OSHW-Logo2_9.8x8mm_SilkScreen, Symbols:OSHW-Logo2_9.8x8mm_SilkScreen, F.Cu at (117.0, 105.5)
Other:
- board text added: "CE"
- board text added: "CSN"
- board text added: "IRQ"
- board text added: "TAPR OHL tapr.org/ohl"
- board text added: "wFM-Tx 0.1 calcium3000.wordpress.com"
- board text removed: "CHARGE"
